Commit message: change robot color

File: Assignment3/ros_gazebo_rviz/urdf/robot_tutorial.xacro (robot description, xacro)
@@ -22,4 +22,7 @@
   <material name="red">
     <color rgba="0.8 0.0 0.0 1.0"/>
+  </material>
+  <material name="green">
+    <color rgba="0.0 0.8 0.0 1.0"/>
   </material>
   <!--Interial macros-->
@@ -81,5 +84,5 @@
           <cylinder radius="${wheel_radius}" length="0.005"/>
         </geometry>
-        <material name="red"/>
+        <material name="green"/>
       </visual>
       <collision>

Commit message: fix sensor size

File: Assignment3/ros_gazebo_rviz/urdf/robot_tutorial.xacro (robot description, xacro)
@@ -128,12 +128,12 @@
     <origin xyz="${caster_wheel_joint_offset} 0 -${caster_wheel_radius+0.005}" rpy="0 0 0"/>
   </joint>
-  <xacro:include filename="$(find ros_101_gazebo_rviz)/urdf/robot_tutorial_gazebo.xacro"/>
   <!--Laser Joint -->
   <joint name="laser_joint" type="fixed">
       <axis xyz="0 1 0" />
-      <origin xyz="0.075 0 0.2" rpy="0 0 0" />
+      <origin xyz="0.075 0 0.02" rpy="0 0 0" />
       <parent link="base_link" />
       <child link="laser_link" />
   </joint>
+  <xacro:include filename="$(find ros_101_gazebo_rviz)/urdf/robot_tutorial_gazebo.xacro"/>
   <!--Laser Link -->
   <link name="laser_link">
