Commit message: make the wheels green

File: Assignment3/ros_gazebo_rviz/urdf/robot_tutorial_gazebo.xacro (robot description, xacro)
@@ -21,8 +21,8 @@
   </gazebo>
   <gazebo reference="left_wheel">
-    <material>Gazebo/Red</material>
+    <material>Gazebo/Green</material>
   </gazebo>
   <gazebo reference="right_wheel">
-    <material>Gazebo/Red</material>
+    <material>Gazebo/Green</material>
   </gazebo>
 </robot>

Commit message: Start code for auto follow

File: Assignment3/ros_gazebo_rviz/urdf/robot_tutorial_gazebo.xacro (robot description, xacro)
@@ -56,3 +56,6 @@
     <material>Gazebo/Green</material>
   </gazebo>
+  <gazebo reference="laser_link">
+    <material>Gazebo/Green</material>
+  </gazebo>
 </robot>
